File: KiCADv5_02_files_Validated/TAS3251JMF_MCU_Clean_Ref_KiCADv5_02/untitled.kicad_sch (KiCad schematic)
At the start: 8 parts, among them J14 USB_C_Receptacle_USB2.0_14P, U4 ESP32-S3-WROOM-1, U6 USBLC6-2SC6

Commit message: Minor changes
Connections:
- net GND: now also J14.S1 (SHIELD)
- net VCC_5V: now also C73.1
- net at J14.A5 (CC1), R29.1: no longer C73.1
Other:
- moved on the sheet: C73, R29
Changed lines of the file:
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@@
-	)
-	(junction
-		(at 177.8 29.21)
-		(diameter 0)
-		(color 0 0 0 0)
 	)
 	(junction
@@
 	)
 	(junction
+		(at 123.19 62.23)
+		(diameter 0)
+		(color 0 0 0 0)
+	)
+	(junction
 		(at 138.43 39.37)
 		(diameter 0)
@@
 		(color 0 0 0 0)
 	)
+	(junction
+		(at 189.23 24.13)
+		(diameter 0)
+		(color 0 0 0 0)
+	)
 	(wire
 		(pts
@@
 	(wire
 		(pts
-			(xy 149.86 24.13) (xy 193.04 24.13)
+			(xy 149.86 24.13) (xy 189.23 24.13)
 		)
 		(stroke
@@
 	(wire
 		(pts
-			(xy 138.43 29.21) (xy 177.8 29.21)
+			(xy 177.8 29.21) (xy 138.43 29.21)
 		)
 		(stroke
@@
 	(wire
 		(pts
-			(xy 177.8 29.21) (xy 189.23 29.21)
+			(xy 189.23 24.13) (xy 189.23 31.75)
 		)
 		(stroke
@@
 	(wire
 		(pts
+			(xy 189.23 24.13) (xy 193.04 24.13)
+		)
+		(stroke
+			(width 0)
+			(type default)
+		)
+	)
+	(wire
+		(pts
+			(xy 177.8 31.75) (xy 177.8 29.21)
+		)
+		(stroke
+			(width 0)
+			(type default)
+		)
+	)
+	(wire
+		(pts
 			(xy 160.02 93.98) (xy 160.02 39.37)
+		)
+		(stroke
+			(width 0)
+			(type default)
+		)
+	)
+	(wire
+		(pts
+			(xy 115.57 62.23) (xy 123.19 62.23)
 		)
 		(stroke
@@
 	(symbol
 		(lib_id "Device:CP")
-		(at 189.23 33.02 0)
+		(at 189.23 35.56 0)
 		(unit 1)
 		(exclude_from_sim no)
@@
 		(dnp no)
 		(property "Reference" "C73"
-			(at 192.151 31.8516 0)
+			(at 192.151 34.3916 0)
 			(effects
 				(font
@@
 		)
 		(property "Value" "10µF"
-			(at 192.151 34.163 0)
+			(at 192.151 36.703 0)
 			(effects
 				(font
@@
 		)
 		(property "Footprint" "Capacitor_SMD:CP_Elec_4x5.8"
-			(at 190.1952 36.83 0)
+			(at 190.1952 39.37 0)
 			(effects
 				(font
@@
 		)
 		(property "Datasheet" "xxSMD-ECAP-4x5.3xCAP,AL, 10 μF, 16 V, ±20%,1.35Ω, SMD"
-			(at 189.23 33.02 0)
+			(at 189.23 35.56 0)
 			(effects
 				(font
@@
 		)
 		(property "Description" ""
-			(at 189.23 33.02 0)
+			(at 189.23 35.56 0)
 			(effects
 				(font
@@
 		)
 		(property "Manufacturer" "Panasonic"
-			(at 134.62 148.59 0)
+			(at 134.62 151.13 0)
 			(effects
 				(font
@@
 		)
 		(property "PartNumber" "EEE-FK1C100R"
-			(at 134.62 148.59 0)
+			(at 134.62 151.13 0)
 			(effects
 				(font
@@
 		)
 		(property "Value2" "x16V"
-			(at 134.62 148.59 0)
+			(at 134.62 151.13 0)
 			(effects
 				(font
@@
 		)
 		(property "Manufacturer_Name" "VE-100M1ETR-0405"
-			(at 134.62 148.59 0)
+			(at 134.62 151.13 0)
 			(effects
 				(font
@@
 		)
 		(property "Manufacturer_Part_Number" "C134721"
-			(at 134.62 148.59 0)
+			(at 134.62 151.13 0)
 			(effects
 				(font
@@
 	(symbol
 		(lib_id "power:GND")
-		(at 177.8 36.83 0)
+		(at 177.8 39.37 0)
 		(unit 1)
 		(exclude_from_sim no)
@@
 		(fields_autoplaced yes)
 		(property "Reference" "#PWR020"
-			(at 177.8 43.18 0)
+			(at 177.8 45.72 0)
 			(effects
 				(font
@@
 		)
 		(property "Value" "GND"
-			(at 177.8 41.91 0)
+			(at 177.8 44.45 0)
 			(effects
 				(font
@@
 		)
 		(property "Footprint" ""
-			(at 177.8 36.83 0)
+			(at 177.8 39.37 0)
 			(effects
 				(font
@@
 		)
 		(property "Datasheet" ""
-			(at 177.8 36.83 0)
+			(at 177.8 39.37 0)
 			(effects
 				(font
@@
 		)
 		(property "Description" "Power symbol creates a global label with name \"GND\" , ground"
-			(at 177.8 36.83 0)
+			(at 177.8 39.37 0)
 			(effects
 				(font
@@
 	(symbol
 		(lib_id "Device:R")
-		(at 177.8 33.02 0)
+		(at 177.8 35.56 0)
 		(unit 1)
 		(exclude_from_sim no)
@@
 		(fields_autoplaced yes)
 		(property "Reference" "R29"
-			(at 180.34 31.7499 0)
+			(at 180.34 34.2899 0)
 			(effects
 				(font
@@
 		)
 		(property "Value" "5k1"
-			(at 180.34 34.2899 0)
+			(at 180.34 36.8299 0)
 			(effects
 				(font
@@
 		)
 		(property "Footprint" ""
-			(at 176.022 33.02 90)
+			(at 176.022 35.56 90)
 			(effects
 				(font
@@
 		)
 		(property "Datasheet" "~"
-			(at 177.8 33.02 0)
+			(at 177.8 35.56 0)
 			(effects
 				(font
@@
 		)
 		(property "Description" "Resistor"
-			(at 177.8 33.02 0)
+			(at 177.8 35.56 0)
 			(effects
 				(font
@@
 	(symbol
 		(lib_id "power:GND")
-		(at 189.23 36.83 0)
+		(at 189.23 39.37 0)
 		(unit 1)
 		(exclude_from_sim no)
@@
 		(fields_autoplaced yes)
 		(property "Reference" "#PWR024"
-			(at 189.23 43.18 0)
+			(at 189.23 45.72 0)
 			(effects
 				(font
@@
 		)
 		(property "Value" "GND"
-			(at 189.23 41.91 0)
+			(at 189.23 44.45 0)
 			(effects
 				(font
@@
 		)
 		(property "Footprint" ""
-			(at 189.23 36.83 0)
+			(at 189.23 39.37 0)
 			(effects
 				(font
@@
 		)
 		(property "Datasheet" ""
-			(at 189.23 36.83 0)
+			(at 189.23 39.37 0)
 			(effects
 				(font
@@
 		)
 		(property "Description" "Power symbol creates a global label with name \"GND\" , ground"
-			(at 189.23 36.83 0)
-			(effects
-				(font
+			(at 189.23 39.37 0)
+			(effects
+				(font
